File: pcb/connector_pcb/connector_pcb.kicad_pcb (KiCad board)
At the start: 2 copper layers, 61.6 x 13 mm, 6 parts

Commit message: update
Parts:
- removed the REF** at (61.7, 116.8)
- removed the REF** at (33.5, 116.1)
- removed the REF** at (84.6, 116.1)
- removed the REF** at (89.5, 113.0)
- added REF**: PinSocket_1x07_P2.54mm_Vertical, Connector_PinSocket_2.54mm:PinSocket_1x07_P2.54mm_Vertical, F.Cu at (78.2, 47.6)
- REF**: value . -> JST_EH_B2B-EH-A_1x02_P2.50mm_Vertical
- moved REF** 52.3 mm to (77.0, 65.4)
- moved REF** 51.0 mm to (36.0, 65.4)
Routing:
- net (no net): track 127.7 -> 258.0 mm
Other:
- board size 61.6 x 13 mm -> 70.7 x 25.4 mm

Commit message: update
Parts:
- added REF**: SolderWirePad_1x01_Drill0.8mm, Connector_Wire:SolderWirePad_1x01_Drill0.8mm, F.Cu at (88.5, 57.1)
- added REF**: SolderWirePad_1x01_Drill0.8mm, Connector_Wire:SolderWirePad_1x01_Drill0.8mm, F.Cu at (37.7, 57.1)
- added REF**: SolderWirePad_1x01_Drill0.8mm, Connector_Wire:SolderWirePad_1x01_Drill0.8mm, F.Cu at (37.7, 60.1)
- added REF**: SolderWirePad_1x01_Drill0.8mm, Connector_Wire:SolderWirePad_1x01_Drill0.8mm, F.Cu at (88.5, 60.1)
- added REF**: SolderWirePad_1x01_Drill0.8mm, Connector_Wire:SolderWirePad_1x01_Drill0.8mm, F.Cu at (81.8, 57.4)
- moved REF** 5.36 mm to (78.1, 53.0)
Routing:
- net (no net): track 258.0 -> 247.0 mm
Other:
- outline, holes or cut-outs redrawn
