File: pcb/main/pcb.kicad_pcb (KiCad board)
At the start: 2 copper layers, 71.1 x 54.6 mm, 21 parts, among them U1 L293D, m3_schraube ., m3_schraube 0.8mm

Commit message: update
Parts:
- removed the REF** at (67.9, 87.6)
- removed the REF** at (77.5, 71.8)
- added display_abstandshalter_m3_unten_senkkopf: ., Connector_Wire:SolderWirePad_1x01_Drill0.8mm, F.Cu at (71.1, 47.2)
- moved zugentlastung_usb-pwrbnk 23.3 mm to (59.7, 64.8)
- moved REF** 22.9 mm to (69.8, 64.8)
- moved REF** 21.6 mm to (61.0, 43.2)
- moved REF** 21.6 mm to (74.9, 74.9), turned to 270 degrees
- moved REF** 12.7 mm to (71.1, 55.9), turned to 180 degrees
- moved REF** 6.35 mm to (124.5, 86.4)
- moved m3_schraube 5.46 mm to (76.6, 43.2)
Connections:
- REF** pad 1: mot_- -> (no net)
- REF** pad 2: Net-(U1-Pad4) -> (no net)
- REF** pad 3: mot_+ -> (no net)
- REF** pad 4: end_signal -> (no net)
- REF** pad 5: encoder1_signal -> (no net)
- REF** pad 6: encoder2_signal -> (no net)
- REF** pad 21: (no net) -> end_signal
- REF** pad 8: ardu_gnd2 -> (no net)
Routing:
- net (no net): track 323.5 -> 447.4 mm
- net ardu_gnd2: track 69.2 -> 0.00 mm
- net encoder1_signal: track 23.5 -> 0.00 mm
- net encoder2_signal: track 21.3 -> 0.00 mm
- net mot_-: track 19.1 -> 27.0 mm
- net mot_+: track 16.9 -> 23.5 mm
- net Net-(U1-Pad4): track 16.9 -> 23.5 mm
- net end_signal: track 25.6 -> 32.1 mm
- net ardu_vcc: track 120.1 -> 125.1 mm
- net Net-(A1-Pad9): track 4.07 -> 0.00 mm
Other:
- outline, holes or cut-outs redrawn
- board text added: "slider 2019-2021"
